File: Production Files/T5400_Barometer_Breakout-Panel-v10.brd (EAGLE design)
At the start: 116.8 x 115.3 mm, 363 parts, among them U1 T5400, U10 T5400, U11 T5400, U12 T5400, U13 T5400, U14 T5400, U15 T5400, U16 T5400, U17 T5400, U18 T5400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

Commit message: Recreated Panel
Parts:
- moved E$4 1.27 mm to (112.4, 11.9)
- moved E$5 1.27 mm to (112.4, 103.4)
- moved E$1 0.51 mm to (4.57, 11.2)
Other:
- board text added: "T5403 Barometric Sensor"
- board text removed: "T5400 Barometric Sensor"
