File: Hardware/T5403_Barometer_Breakout.brd (EAGLE design)
At the start: 25.4 x 16.5 mm, 16 parts, among them U1 T5400

Commit message: cleaned up SCH and replaced components with correct Sparkle ID's
Parts:
- R1, R2: device SparkFun-Passives:0603-RES -> SparkFun-Resistors:0603
- R3, R4: device SparkFun-Passives:0603-RES -> SparkFun-Resistors:0603-RES
- U1: device T5400:T5400 -> SparkFun-Sensors:T5400
Changed lines of the file:
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@@
 </autorouter>
 <elements>
-<element name="U1" library="T5400" package="T5400" value="T5400" x="13.97" y="10.414" rot="R90"/>
+<element name="U1" library="SparkFun-Sensors" package="T5400" value="T5400" x="13.97" y="10.414" rot="R90">
+<attribute name="PROD_ID" value="IC-11772" x="13.97" y="10.414" size="1.778" layer="27" rot="R90" display="off"/>
+</element>
 <element name="JP1" library="SparkFun-Connectors" package="1X08" value="" x="3.81" y="1.27" smashed="yes">
 <attribute name="NAME" x="2.2352" y="1.1938" size="0.8128" layer="25" font="vector" ratio="15" rot="R90"/>
@@
 <element name="FRAME1" library="SparkFun-Aesthetics" package="CREATIVE_COMMONS" value="FRAME-LETTER" x="0" y="-8.89"/>
 <element name="LOGO2" library="SparkFun-Aesthetics" package="OSHW-LOGO-S" value="OSHW-LOGOS" x="21.844" y="8.382"/>
-<element name="R1" library="SparkFun-Passives" package="0603-RES" value="4.7k" x="9.144" y="8.89" rot="R180"/>
-<element name="R2" library="SparkFun-Passives" package="0603-RES" value="4.7k" x="9.144" y="10.922" rot="R180"/>
+<element name="R1" library="SparkFun-Resistors" package="0603" value="4.7k" x="9.144" y="8.89" rot="R180">
+<attribute name="PROD_ID" value="RES-07857" x="9.144" y="8.89" size="1.778" layer="27" rot="R180" display="off"/>
+</element>
+<element name="R2" library="SparkFun-Resistors" package="0603" value="4.7k" x="9.144" y="10.922" rot="R180">
+<attribute name="PROD_ID" value="RES-07857" x="9.144" y="10.922" size="1.778" layer="27" rot="R180" display="off"/>
+</element>
 <element name="C1" library="SparkFun-Capacitors" package="0603-CAP" value=".1uF" x="13.97" y="7.366" rot="R180">
 <attribute name="PROD_ID" value="CAP-08604" x="13.97" y="7.366" size="1.778" layer="27" rot="R180" display="off"/>
@@
 <element name="STANDOFF2" library="SparkFun-Electromechanical" package="STAND-OFF" value="STAND-OFF" x="22.86" y="13.97"/>
 <element name="LOGO1" library="SparkFun-Aesthetics" package="SFE-NEW-WEBLOGO" value="LOGO-SFENEW" x="22.352" y="7.366" rot="MR0"/>
-<element name="R3" library="SparkFun-Passives" package="0603-RES" value="10k" x="9.144" y="12.954" rot="R180"/>
+<element name="R3" library="SparkFun-Resistors" package="0603-RES" value="10k" x="9.144" y="12.954" rot="R180">
+<attribute name="PROD_ID" value="RES-00824" x="9.144" y="12.954" size="1.778" layer="27" rot="R180" display="off"/>
+<attribute name="VALUE" value="10K" x="9.144" y="12.954" size="1.778" layer="27" rot="R180" display="off"/>
+</element>
 <element name="FID1" library="SparkFun-Aesthetics" package="FIDUCIAL-1X2" value="FIDUCIAL1X2" x="1.27" y="11.43"/>
 <element name="FID2" library="SparkFun-Aesthetics" package="FIDUCIAL-1X2" value="FIDUCIAL1X2" x="24.13" y="2.54"/>
 <element name="LOGO3" library="SparkFun-Aesthetics" package="SFE_LOGO_FLAME_.1" value="SFE_LOGO_FLAME.1_INCH" x="1.524" y="6.858"/>
 <element name="SJ2" library="SparkFun-Passives" package="SJ_3_PASTE1&amp;2&amp;3" value="" x="6.35" y="9.906" rot="R90"/>
-<element name="R4" library="SparkFun-Passives" package="0603-RES" value="10k" x="17.018" y="7.874" rot="R90"/>
+<element name="R4" library="SparkFun-Resistors" package="0603-RES" value="10k" x="17.018" y="7.874" rot="R90">
+<attribute name="PROD_ID" value="RES-00824" x="17.018" y="7.874" size="1.778" layer="27" rot="R90" display="off"/>
+<attribute name="VALUE" value="10K" x="17.018" y="7.874" size="1.778" layer="27" rot="R90" display="off"/>
+</element>
 </elements>
 <signals>
